File: Reference_Designs/SingleDryCell-LR6|AA/SingleDryCell.kicad_sch (KiCad schematic)
At the start: 20 parts, among them J7 MDT420E01001, Q1 Q_NPN_BCE

Commit message: Release Rev B of reference design.
Parts:
- removed BAT1: LR6/AA x4, symbol blues-kicad-lib:Battery
- removed C1: 47µF, symbol Device:C_Polarized
- removed D1: D_Zener_Filled, symbol Device:D_Zener_Filled
- removed LDO-1: ~, symbol Regulator_Linear:AP2204R-3.3
- removed R (x2): 100, symbol Device:R_US
- added BUCK, SCOOP: ~, symbol Regulator_Linear:AP2204R-3.3
- added C1: 100nF, symbol Device:C_Small
- added D1, D10, D11, D12, D13, D14, D15, D16, D2, D3, D4, D5, D6, D7, D8, D9: D_Small_Filled, symbol Device:D_Small_Filled
- added J1: USB, symbol Connector:USB_B
- added R10, R11, R12, R5, R6, R7, R8, R9: 200, symbol Device:R_US
- added TP1: AUX_EN, symbol Connector:TestPoint
- added TP2: AUX_RX, symbol Connector:TestPoint
- added TP3: AUX_TX, symbol Connector:TestPoint
- R1: value 100 -> 0R
- R2: value 100 -> NU
- renumbered LDO-2 to BOOST, C4 to C2, C6 to C2, C2 to C4, J7 to J2, R3 to R10, R4 to R13, R5 to R3, R6 to R4
Connections:
- net +BATT: now also R10.1, BUCK.1 (VIN), SCOOP.3 (OUT-)
- net AUX1: now also MCU.23 (GPIO2)
- net AUX2: now also MCU.22 (GPIO3)
- net AUX3: now also MCU.21 (GPIO4)
- net AUX4: now also MCU.20 (GPIO5)
- net Earth: now also BUCK.2 (GND), C1.2, D10.2 (A), D11.2 (A), D12.2 (A), D13.2 (A), D14.2 (A), D15.2 (A), D16.2 (A), D9.2 (A), J1.4 (GND), SCOOP.3 (OUT-)
- net RX: now also D15.1 (K), D7.2 (A), R11.2
- net SCL: now also D1.2 (A), D9.1 (K), R5.2
- net SDA: now also D10.1 (K), D2.2 (A), R6.2
- net TX: now also D16.1 (K), D8.2 (A), R12.2
- net VCC: now also R1.2, R2.2
- net at MCU.15 (RXD): now also R12.1; no longer R2.1
- net at J2.13 (VUSB): now also C1.1, J1.1 (VBUS)
- net at J2.56 (AUX_EN_P): now also D12.1 (K), D4.2 (A), R8.2
- net at J2.58 (AUX_RX_P): now also D13.1 (K), D5.2 (A), R9.2
- net at J2.60 (AUX_TX_P): now also D14.1 (K), D6.2 (A), R10.2
- net at J2.7 (USB_DP): now also J1.3 (D+)
- net at J2.9 (USB_DM): now also J1.2 (D-)
- net at MCU.14 (TXD): now also R11.1; no longer R1.1
- net at MCU.17 (SDA): now also R6.1
- net at MCU.18 (SCL): now also R5.1
- net +3V3: now reaches BOOST.3 (VOUT), MCU.2 (VCC)
- net +3V3: now also R1.1, D1.1 (K), D2.1 (K), D3.1 (K), D4.1 (K), D5.1 (K), D6.1 (K), D7.1 (K), D8.1 (K)
- net +1V8: now reaches BOOST.1 (VIN)
- net +1V8: now also R2.1, BUCK.3 (VOUT); no longer R10.1
- net ATTN/1.2C renamed ATTN
- net ATTN: now also D11.1 (K), D3.2 (A), R7.2
- new net: MCU.19 (GPIO6), R7.1
- new net: R9.1, TP2.1
- new net: R8.1, TP1.1
- new net: R10.1, TP3.1
Other:
- note added: "2.5V-3.8V"
- note added: "Low Power Design Application Note - Reference Diagram"
- note added: "Note: I2C 10kΩ pullups are on actual Notecard"
- note added: "Note: If VIO is supplied with 1.8V, level shifting is required in the Protection block."
- note added: "Power Supply"
- note added: "Protection & Termination"
- note added: "Supply 4.8V to 24V. USB compatible."
- note added: "VIO Supply"
- note removed: "3.3V"
- note removed: "3.6V"
- note removed: "Level shifter or protection req."
- note removed: "Note: AUX pins broken out to test points AND/OR header vias"
- note removed: "Note: i2c 10k pullups on actual Notecard"
- note removed: "Reference Design of a Single Dry Cell LR6/AA"
- note removed: "SWITCHED"
- moved on the sheet: C2, C3, C4, J2, R3, R4
